Commit message: tes env

File: config/urdf/abb_cell.urdf (robot description, URDF)
Before this commit: robot combined, 34 links, 33 joints
Links:
- removed link ABB_1200_5_90_base_link
- removed link ABB_1200_5_90_link_1
- removed link ABB_1200_5_90_link_2
- removed link ABB_1200_5_90_link_3
- removed link ABB_1200_5_90_link_4
- removed link ABB_1200_5_90_link_5
- removed link ABB_1200_5_90_link_6
- removed link ABB_1200_5_90_pedestal
- removed link FANUC_lrmate200id_base_link
- removed link FANUC_lrmate200id_link_1
- removed link FANUC_lrmate200id_link_2
- removed link FANUC_lrmate200id_link_3
- removed link FANUC_lrmate200id_link_4
- removed link FANUC_lrmate200id_link_5
- removed link FANUC_lrmate200id_link_6
- removed link FANUC_m10ia_base_link
- removed link FANUC_m10ia_link_1
- removed link FANUC_m10ia_link_2
- removed link FANUC_m10ia_link_3
- removed link FANUC_m10ia_link_4
- removed link FANUC_m10ia_link_5
- removed link FANUC_m10ia_link_6
- removed link FANUC_m10ia_tool
- removed link curve_1_base_link
- removed link curve_2_base_link
- added link ABB_1200_5_90; collision box size=1 1 3; visual box size=1 1 3
Joints:
- removed joint ABB_1200_5_90_joint_1
- removed joint ABB_1200_5_90_joint_2
- removed joint ABB_1200_5_90_joint_3
- removed joint ABB_1200_5_90_joint_4
- removed joint ABB_1200_5_90_joint_5
- removed joint ABB_1200_5_90_joint_6
- removed joint ABB_1200_5_90_pedestal_JOINT_0
- removed joint FANUC_lrmate200id_joint_1
- removed joint FANUC_lrmate200id_joint_2
- removed joint FANUC_lrmate200id_joint_3
- removed joint FANUC_lrmate200id_joint_4
- removed joint FANUC_lrmate200id_joint_5
- removed joint FANUC_lrmate200id_joint_6
- removed joint FANUC_lrmate200id_pose
- removed joint FANUC_m10ia_joint_1
- removed joint FANUC_m10ia_joint_2
- removed joint FANUC_m10ia_joint_3
- removed joint FANUC_m10ia_joint_4
- removed joint FANUC_m10ia_joint_5
- removed joint FANUC_m10ia_joint_6
- removed joint FANUC_m10ia_joint_6-tool0
- removed joint FANUC_m10ia_pose
- removed joint curve_1_pose
- removed joint curve_2_pose
- joint ABB_1200_5_90_pose: child ABB_1200_5_90_pedestal -> ABB_1200_5_90; origin xyz=0 5.0 5.0 rpy=0.0 0.0 0.0 -> xyz=1 1 0 rpy=0.0 0.0 0.0
- joint ABB_6640_180_255_pose: origin xyz=5.0 0 5.0 rpy=0.0 0.0 0.0 -> xyz=0 0 0 rpy=0.0 0.0 0.0

Commit message: abb cell tess env

File: config/urdf/abb_cell.urdf (robot description, URDF)
Before this commit: robot combined, 10 links, 9 joints
Links:
- removed link ABB_1200_5_90
- added link ABB_6640_180_255_pedestal; collision box size=1.2192 1.0668 0.0254; visual box size=1.2192 1.0668 0.0254
- added link Shelf1; collision box size=1.0668 0.7366 2; visual box size=1.0668 0.7366 2
- added link Shelf2; collision box size=0.508 1.143 2.286; visual box size=0.508 1.143 2.286
- added link Table1; collision box size=0.90805 1.905 1.32; visual box size=0.90805 1.905 1.32
- added link Table2; collision box size=0.6096 1.2192 0.7112; visual box size=0.6096 1.2192 0.7112
- added link Wall1; collision box size=0.01 6.4 4; visual box size=0.01 6.4 4
- added link Wall2; collision box size=0.01 6.4 4; visual box size=0.01 6.4 4
- added link Wall3; collision box size=4.953 0.01 4; visual box size=4.953 0.01 4
- added link Wall4; collision box size=4.953 0.01 4; visual box size=4.953 0.01 4
Joints:
- removed joint ABB_1200_5_90_pose
- added joint ABB_6640_180_255_pedestal_joint: type fixed, parent ABB_6640_180_255_base_link, child ABB_6640_180_255_pedestal, origin xyz=0 0 0 rpy=0.0 0.0 0.0
- added joint Table1_pose: type fixed, parent world, child Table1, origin xyz=-0.542925 1.6637 0.66 rpy=0.0 0.0 0
- added joint Table2_pose: type fixed, parent world, child Table2, origin xyz=0.2159 2.0066 0.3556 rpy=0.0 0.0 0
- added joint Wall1_pose: type fixed, parent world, child Wall1, origin xyz=-1.1303 0 2 rpy=0.0 0.0 0
- added joint Wall2_pose: type fixed, parent world, child Wall2, origin xyz=3.8227 0 2 rpy=0.0 0.0 0
- added joint Wall3_pose: type fixed, parent world, child Wall3, origin xyz=1.3462 -3.2 2 rpy=0.0 0.0 0
- added joint Wall4_pose: type fixed, parent world, child Wall4, origin xyz=1.3462 3.2 2 rpy=0.0 0.0 0
- added joint shelf1_pose: type fixed, parent world, child Shelf1, origin xyz=-0.0635 -2.6797 1 rpy=0.0 0.0 0
- added joint shelf2_pose: type fixed, parent world, child Shelf2, origin xyz=3.3528 -2.0193 1.1143 rpy=0.0 0.0 0
- joint ABB_6640_180_255_pose: origin xyz=0 0 0 rpy=0.0 0.0 0.0 -> xyz=0 0 0.0254 rpy=0.0 0.0 0.0

Commit message: abb cell env sim test

File: config/urdf/abb_cell.urdf (robot description, URDF)
Before this commit: robot combined, 18 links, 17 joints
Links:
- removed link ABB_6640_180_255_tool
- added link Ground; collision box size=4.953 6.4 0.01; visual box size=4.953 6.4 0.01
Joints:
- removed joint joint_6-tool0
- added joint Ground_pose: type fixed, parent world, child Ground, origin xyz=1.3462 0 -0.005 rpy=0.0 0.0 0
- joint ABB_6640_180_255_pedestal_joint: origin xyz=0 0 0 rpy=0.0 0.0 0.0 -> xyz=0 0 -0.0127 rpy=0.0 0.0 0.0
- joint shelf2_pose: origin xyz=3.3528 -2.0193 1.1143 rpy=0.0 0.0 0 -> xyz=3.3528 -2.0193 1.143 rpy=0.0 0.0 0
