Commit message: motoman acc

File: config/urdf/motoman_cell.urdf (robot description, URDF)
Before this commit: robot combined, 30 links, 29 joints
Links:
- added link MA2010_filler; collision box size=0.3 0.5 0.3; visual box size=0.4 0.2 0.3
Joints:
- added joint filler_joint: type fixed, parent MA2010_link_2_l, child MA2010_filler, origin xyz=0.0 -0.36 0.4 rpy=0 0 0, axis 0 0 0

Commit message: acc capture motoman

File: config/urdf/motoman_cell.urdf (robot description, URDF)
Before this commit: robot combined, 31 links, 30 joints
Links:
- added link Ground; collision box size=4.953 6.4 0.01; visual box size=4.953 6.4 0.01
Joints:
- added joint Ground_pose: type fixed, parent world, child Ground, origin xyz=1.3462 0 -0.005 rpy=0.0 0.0 0
- joint MA1440_pose: origin xyz=4 0 0.908 rpy=0.0 0.0 3.14159 -> xyz=2.689552 -0.39515 0.908 rpy=0.0 0.0 3.14159

Commit message: new exp

File: config/urdf/motoman_cell.urdf (robot description, URDF)
Before this commit: robot combined, 32 links, 31 joints
Links:
- link MA2010_pedestal: geometry collision box size=0.75 0.6858 0.762; visual box size=0.75 0.6858 0.762

Commit message: ma1440 test

File: config/urdf/motoman_cell.urdf (robot description, URDF)
Before this commit: robot combined, 32 links, 31 joints
Links:
- removed link MA1440_tool0
- added link Wall1; collision box size=0.01 6.4 4; visual box size=0.01 6.4 4
- added link scanner; collision box size=0.3 0.2 0.2; visual box size=0.3 0.2 0.2
Joints:
- removed joint MA1440_joint_6_t-tool0
- added joint Wall1_pose: type fixed, parent world, child Wall1, origin xyz=3.44 0 2 rpy=0.0 0.0 0
- added joint scanner_joint: type fixed, parent MA1440_link_6_t, child scanner, origin xyz=0.25 0 0 rpy=0 0 0, axis 0 0 0

Commit message: scanner update

File: config/urdf/motoman_cell.urdf (robot description, URDF)
Before this commit: robot combined, 33 links, 32 joints
Links:
- link scanner: geometry collision box size=0.3 0.2 0.25; visual box size=0.3 0.2 0.25
Joints:
- joint scanner_joint: origin xyz=0.25 0 0 rpy=0 0 0 -> xyz=0.25 0 -0.05 rpy=0 0 0

Commit message: urdf updates

File: config/urdf/motoman_cell.urdf (robot description, URDF)
Before this commit: robot combined, 33 links, 32 joints
Links:
- removed link weldgun
- added link torch; collision mesh filename=model://MA_2010_A0/meshes/collision/torch.stl scale=0.001 0.001 0.001; visual mesh filename=model://MA_2010_A0/meshes/visual/torch.stl scale=0.001 0.001 0.001
Joints:
- removed joint weldgun_joint
- added joint torch_joint: type fixed, parent MA2010_link_6_t, child torch, origin xyz=0.1 0 0 rpy=0 1.57 0, axis 0 0 0
